File: powerplay/powerplay.kicad_pcb (KiCad board)
At the start: 2 copper layers, 62 x 30 mm, 31 parts, among them J1 USB_C_Receptacle, J2 Jack-DC, J3 Jack-DC, Q1 DMN3009SFG-7, Q2 DMN3009SFG-7, U2 TSR_1-2412

Commit message: updated
Parts:
- U1: value ~ -> AP33771C
Changed lines of the file:
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@@
       (sketchpadsonfab false)
       (subtractmaskfromsilk false)
-      (outputformat 4)
+      (outputformat 1)
       (mirror false)
       (drillshape 0)
       (scaleselection 1)
-      (outputdirectory "PDFs/")
+      (outputdirectory "fabrication/")
     )
   )
@@
         (effects (font (size 1 1) (thickness 0.15)))
     )
-    (fp_text value "~" (at 0 2.55 90) (layer "F.Fab")
-        (effects (font (size 1 1) (thickness 0.15)))
-    )
+    (fp_text value "AP33771C" (at 0 2.55 90) (layer "F.Fab")
+        (effects (font (size 1 1) (thickness 0.15)))
+    )
