File: powerplay/powerplay.kicad_sch (KiCad schematic)
At the start: 31 parts, among them J1 USB_C_Receptacle, J2 Jack-DC, J3 Jack-DC, Q1 DMN3009SFG-7, Q2 DMN3009SFG-7, U2 TSR_1-2412

Commit message: updated
Parts:
- U1: value ~ -> AP33771C
Changed lines of the file:
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@@
   )
   (symbol (lib_id "SamacSys_Parts:AP33771C") (at 140.97 82.55 0) (unit 1)
-    (in_bom yes) (on_board yes) (dnp no) (fields_autoplaced)
+    (in_bom yes) (on_board yes) (dnp no)
     (property "Reference" "U1" (at 150.495 55.88 0)
       (effects (font (size 1.27 1.27)))
     )
-    (property "Value" "~" (at 140.97 73.66 0)
+    (property "Value" "AP33771C" (at 148.59 82.55 0)
       (effects (font (size 1.27 1.27)))
     )
